File: pcb/Starbie.kicad_sch (KiCad schematic)
At the start: 11 parts, among them J1 Conn_01x04_Pin, J2 Conn_01x08_Pin, SW1 SW_Push, SW2 SW_Push, U1 DHT11, U2 XIAO-ESP32-C3-SMD

Commit message: Refactor LED properties and update designators in PCB and schematic files
Parts:
- D1: symbol Device:LED_RGBA -> Device:LED_RAGB
Connections:
- net +3.3V: now also D1.2 (A); no longer D1.4 (A)
- net at R3.2: now also D1.3 (GK); no longer D1.2 (GK)
- net at R4.2: now also D1.4 (BK); no longer D1.3 (BK)
Changed lines of the file:
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@@
 	)
 	(symbol
-		(lib_id "Device:LED_RGBA")
+		(lib_id "Device:LED_RAGB")
 		(at 39.37 93.98 0)
 		(unit 1)
@@
 			)
 		)
-		(property "Description" "RGB LED, red/green/blue/anode"
+		(property "Description" "RGB LED, red/anode/green/blue"
 			(at 39.37 93.98 0)
 			(hide yes)
